File: PCB/hackpad.kicad_sch (KiCad schematic)
At the start: 9 parts, among them SW1 SW_Push, SW2 SW_Push, SW3 SW_Push, SW4 SW_Push, SW5 SW_Push, SW7 SW_Push, U1 XIAO-RP2040-DIP

Commit message: update pcb + schematic to not short the entire board (...oops)
readme update soon
Connections:
- net at SW5.2: now also U1.6 (GPIO7/SCL); no longer U1.12 (3V3)
Changed lines of the file:
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@@
-	(wire
-		(pts
-			(xy 133.35 153.67) (xy 133.35 119.38)
-		)
-		(stroke
-			(width 0)
-			(type default)
-		)
-	)
 	(wire
 		(pts
@@
 	(wire
 		(pts
-			(xy 113.03 134.62) (xy 177.8 134.62)
-		)
-		(stroke
-			(width 0)
-			(type default)
-		)
-	)
-	(wire
-		(pts
 			(xy 102.87 109.22) (xy 102.87 120.65)
 		)
@@
 	(wire
 		(pts
-			(xy 177.8 134.62) (xy 177.8 104.14)
+			(xy 132.08 143.51) (xy 132.08 115.57)
 		)
 		(stroke
@@
 	(wire
 		(pts
-			(xy 113.03 143.51) (xy 113.03 134.62)
+			(xy 113.03 143.51) (xy 132.08 143.51)
 		)
 		(stroke
@@
 	(wire
 		(pts
-			(xy 168.91 104.14) (xy 177.8 104.14)
+			(xy 133.35 119.38) (xy 133.35 153.67)
 		)
 		(stroke
@@
 		)
 		(stroke
+			(width 0)
+			(type default)
+		)
+	)
+	(wire
+		(pts
+			(xy 132.08 115.57) (xy 133.35 115.57)
+		)
+		(stroke
